Commit message: Switched back to fingers fixed

File: schunk_egp40_description/urdf/schunk_egp40.xacro (robot description, xacro)
@@ -107,5 +107,5 @@
             <origin xyz="0.0 0.0 ${body_height/2+base_height}" rpy="0.0 0.0 0.0" />
         </joint>
-        <joint name="${prefix}schunk_egp40_finger_left_joint" type="prismatic">
+        <joint name="${prefix}schunk_egp40_finger_left_joint" type="fixed">
             <parent link="${prefix}schunk_egp40_body_link" />
             <child link="${prefix}schunk_egp40_finger_left_link" />
@@ -116,5 +116,5 @@
             <limit lower="${-body_length/16}" upper="${body_length/16}" velocity="100" effort="100" />
         </joint>
-        <joint name="schunk_egp40_finger_right_joint" type="prismatic">
+        <joint name="schunk_egp40_finger_right_joint" type="fixed">
             <parent link="${prefix}schunk_egp40_body_link" />
             <child link="${prefix}schunk_egp40_finger_right_link" />

Commit message: Integrated joint states

File: schunk_egp40_description/urdf/schunk_egp40.xacro (robot description, xacro)
@@ -107,5 +107,5 @@
             <origin xyz="0.0 0.0 ${body_height/2+base_height}" rpy="0.0 0.0 0.0" />
         </joint>
-        <joint name="${prefix}schunk_egp40_finger_left_joint" type="fixed">
+        <joint name="${prefix}schunk_egp40_finger_left_joint" type="prismatic">
             <parent link="${prefix}schunk_egp40_body_link" />
             <child link="${prefix}schunk_egp40_finger_left_link" />
@@ -116,5 +116,5 @@
             <limit lower="${-body_length/16}" upper="${body_length/16}" velocity="100" effort="100" />
         </joint>
-        <joint name="schunk_egp40_finger_right_joint" type="fixed">
+        <joint name="schunk_egp40_finger_right_joint" type="prismatic">
             <parent link="${prefix}schunk_egp40_body_link" />
             <child link="${prefix}schunk_egp40_finger_right_link" />
